File: kicad/interhardware.kicad_sch (KiCad schematic)
At the start: 0 parts

Commit message: feat(kicad): transcribe Si3050 EVB page 3 schematic
Parts:
- added C1, C2: 33pF, symbol EVB_2PIN
- added C10: 0.01uF, symbol EVB_2PIN
- added C232, R236, R237, R7, R8: NI, symbol EVB_2PIN
- added C3: 3.9nF, symbol EVB_2PIN
- added C30, C31: 120pF, symbol EVB_2PIN
- added C4: 1uF, symbol EVB_2PIN
- added C5, C50, C51, C6: 0.1uF, symbol EVB_2PIN
- added C7: 2.7nF, symbol EVB_2PIN
- added C8, C9: 680pF, symbol EVB_2PIN
- added D1: HD04, symbol EVB_2PIN
- added FB1, FB2, FB203, FB204: 600 Ohm, symbol EVB_2PIN
- added J1: RJ11 LINE, symbol EVB_2PIN
- added Q1, Q3: MMBTA42LT1, symbol EVB_2PIN
- added Q2: MMBTA92LT1, symbol EVB_2PIN
- added Q4, Q5: MMBTA06LT1, symbol EVB_2PIN
- added R1, R12, R13: 56.2, symbol EVB_2PIN
- added R10: 536, symbol EVB_2PIN
- added R11: 73.2, symbol EVB_2PIN
- added R2: 150, symbol EVB_2PIN
- added R3: 3.65K, symbol EVB_2PIN
- added R30: 20, symbol EVB_2PIN
- added R31, R33: 5.1M, symbol EVB_2PIN
- added R32: 15M, symbol EVB_2PIN
- added R4: 2.49K, symbol EVB_2PIN
- added R5, R6: 100K, symbol EVB_2PIN
- added R9: 1M, symbol EVB_2PIN
- added U1: Si3050-FM, symbol EVB_SI3050
- added U2: Si3019-FM, symbol EVB_SI3019
- added V1: P3100SB, symbol EVB_2PIN
- added Z1: 43V, symbol EVB_2PIN
Connections:
- new net AOUT_INT: U1.5 (P5)
- new net C1A: C1.1 (P1), U1.11 (P11)
- new net C1B: R1.2 (P2), U2.13 (P13)
- new net C2A: C2.1 (P1), U1.14 (P14)
- new net C2B: R12.2 (P2), U2.14 (P14)
- new net CS: U1.19 (P19)
- new net DCT: C10.2 (P2), R3.1 (P1), R4.2 (P2), R9.2 (P2)
- new net DCT2: U2.4 (P4)
- new net DCT3: U2.6 (P6)
- new net DRX: U1.15 (P15)
- new net DTX: U1.18 (P18)
- new net FSYNC: U1.20 (P20)
- new net GND: C50.2 (P2), C51.2 (P2), U1.10 (P10)
- new net IB: U2.16 (P16)
- new net IGND: C3.2 (P2), C4.2 (P2), C5.2 (P2), C6.2 (P2), C7.2 (P2), C8.2 (P2), C9.2 (P2), R236.2 (P2), R237.2 (P2), R5.2 (P2), R6.2 (P2), R7.2 (P2), U2.3 (P3)
- new net ISO_C1: C1.2 (P2), R1.1 (P1)
- new net ISO_C2: C2.2 (P2), R12.1 (P1)
- new net LINE_RING: FB1.1 (P1), FB204.2 (P2), V1.2 (P2), Z1.2 (P2)
- new net LINE_TIP: FB2.1 (P1), FB203.2 (P2), V1.1 (P1), Z1.1 (P1)
- new net PCLK: U1.17 (P17)
- new net Q1B: Q1.1 (P1), R5.1 (P1)
- new net Q1E: Q1.2 (P2), R10.1 (P1)
- new net Q2B: Q2.2 (P2), R10.2 (P2)
- new net Q3B: Q3.1 (P1), R6.1 (P1)
- new net Q3E: Q3.2 (P2)
- new net Q4B: Q4.1 (P1), R2.2 (P2), R3.2 (P2)
- new net Q5E: Q5.2 (P2), R11.1 (P1)
- new net QB: Q5.1 (P1), R11.2 (P2), U2.5 (P5)
- new net QE: C10.1 (P1), Q2.1 (P1), R2.1 (P1), R4.1 (P1), R9.1 (P1)
- new net QE2: Q4.2 (P2), U2.8 (P8)
- new net RG: U1.6 (P6)
- new net RGDT: U1.16 (P16)
- new net RING: FB1.2 (P2), J1.2 (P2)
- new net RING_SENSE: C232.1 (P1), C30.2 (P2), D1.2 (P2), FB204.1 (P1), R237.1 (P1), R32.1 (P1)
- new net RNG1: C31.1 (P1), C8.1 (P1), R31.2 (P2), R33.2 (P2), R8.1 (P1), U2.12 (P12)
- new net RNG2: C30.1 (P1), C9.1 (P1), R32.2 (P2), R8.2 (P2), U2.9 (P9)
- new net RST: U1.13 (P13)
- new net RX: C3.1 (P1), R7.1 (P1), U2.15 (P15)
- new net SC: C7.1 (P1), U2.7 (P7)
- new net SCLK: U1.7 (P7)
- new net SDI_THRU: U1.8 (P8)
- new net TGD: U1.4 (P4)
- new net TGDE: U1.3 (P3)
- new net TIP: FB2.2 (P2), J1.1 (P1)
- new net TIP_SENSE: C232.2 (P2), C31.2 (P2), D1.1 (P1), FB203.1 (P1), R236.1 (P1), R31.1 (P1), R33.1 (P1)
- new net VA: C51.1 (P1), R13.1 (P1), U1.12 (P12)
- new net VDD: C50.1 (P1), R13.2 (P2), R30.2 (P2), U1.9 (P9)
- new net VDD_IN: R30.1 (P1)
- new net VREG: C5.1 (P1), C6.1 (P1), U2.11 (P11)
- new net VREG2: C4.1 (P1), U2.10 (P10)
Other:
- note added: "DIGITAL SIDE"
- note added: "ISOLATION BARRIER"
- note added: "LINE SIDE"
- note added: "TELEPHONE LINE"
Changed lines of the file:
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@@
-(kicad_sch
-	(version 20260306)
-	(generator "eeschema")
-	(generator_version "10.0")
-	(paper "A4")
-	(sheet_instances
-		(path "/"
-			(page "1")
-		)
-	)
-	(embedded_fonts no)
-)

Commit message: DAA
Parts:
- removed C1, C2: 33pF, symbol EVB_2PIN
- removed C10: 0.01uF, symbol EVB_2PIN
- removed C232, R236, R237, R7, R8: NI, symbol EVB_2PIN
- removed C3: 3.9nF, symbol EVB_2PIN
- removed C30, C31: 120pF, symbol EVB_2PIN
- removed C4: 1uF, symbol EVB_2PIN
- removed C5, C50, C51, C6: 0.1uF, symbol EVB_2PIN
- removed C7: 2.7nF, symbol EVB_2PIN
- removed C8, C9: 680pF, symbol EVB_2PIN
- removed D1: HD04, symbol EVB_2PIN
- removed FB1, FB2, FB203, FB204: 600 Ohm, symbol EVB_2PIN
- removed J1: RJ11 LINE, symbol EVB_2PIN
- removed Q1, Q3: MMBTA42LT1, symbol EVB_2PIN
- removed Q2: MMBTA92LT1, symbol EVB_2PIN
- removed Q4, Q5: MMBTA06LT1, symbol EVB_2PIN
- removed R1, R12, R13: 56.2, symbol EVB_2PIN
- removed R10: 536, symbol EVB_2PIN
- removed R11: 73.2, symbol EVB_2PIN
- removed R2: 150, symbol EVB_2PIN
- removed R3: 3.65K, symbol EVB_2PIN
- removed R30: 20, symbol EVB_2PIN
- removed R31, R33: 5.1M, symbol EVB_2PIN
- removed R32: 15M, symbol EVB_2PIN
- removed R4: 2.49K, symbol EVB_2PIN
- removed R5, R6: 100K, symbol EVB_2PIN
- removed R9: 1M, symbol EVB_2PIN
- removed U1: Si3050-FM, symbol EVB_SI3050
- removed U2: Si3019-FM, symbol EVB_SI3019
- removed Z1: 43V, symbol EVB_2PIN
- added C1, C2: 33pF, symbol Device:C
- added C10: 0.01uF, symbol Device:C
- added C3: 3.9nF, symbol Device:C
- added C31, C32: 120pF, symbol Device:C
- added C4: 1uF, symbol Device:C
- added C5, C50, C51, C6: 0.1uF, symbol Device:C
- added C7: 2.7nF, symbol Device:C
- added C8, C9: 680pF, symbol Device:C
- added D1: DF04S, Diode_SMD:Diode_Bridge_OnSemi_SDIP-4L, symbol Diode_Bridge:DF04S
- added FB1, FB2, FB203, FB204: 600 Ohm, symbol Device:FerriteBead
- added J2: RJ11, symbol Connector:RJ11
- added Q1, Q3: MMBTA42, Package_TO_SOT_SMD:SOT-23, symbol Transistor_BJT:MMBTA42
- added Q2: MMBTA92, Package_TO_SOT_SMD:SOT-23, symbol Transistor_BJT:MMBTA92
- added Q4, Q5: MMBTA06, Package_TO_SOT_SMD:SOT-23, symbol Transistor_BJT:MMBTA06
- added R1: 1.07k Ohm, symbol Device:R
- added R10: 536 Ohm, symbol Device:R
- added R11: 73.2 Ohm, symbol Device:R
- added R12, R13: 56.2 Ohm, symbol Device:R
- added R2: 150 Ohm, symbol Device:R
- added R3: 3.65k Ohm, symbol Device:R
- added R32, R35: 15M Ohm, symbol Device:R
- added R33, R34: 5.1M Ohm, symbol Device:R
- added R4: 2.49k Ohm, symbol Device:R
- added R5, R6: 100k Ohm, symbol Device:R
- added R52, R53: 47k Ohm, symbol Device:R
- added R9: 1M Ohm, symbol Device:R
- added U1: (no value), symbol interbridge_telephony:SI3019-F-FM
- added U2: (no value), symbol interbridge_telephony:SI3050-E1-FM
- added Z1: 43V, symbol Device:D_Zener
- renumbered V1 to RV1
Connections:
- net LINE_RING is gone; now on net TIP: RV1.2 (P2)
- net LINE_TIP is gone; now on net RING: RV1.1 (P1)
- net GND: now also C50.2, C51.2, C8.2, C9.2, U2.18 (GND), U2.25 (GND_PAD)
- net IGND: now also C3.2, C5.2, C6.2, C7.2, D1.2 (-), R9.2, U1.12 (SC), U1.17 (IGND), U1.21 (IGND_PAD), U1.8 (IGND)
- net RING: now also FB203.2, J2.2
- net TIP: now also FB204.2, J2.1
- net VDD: now also C50.1, R52.1, R53.1, U2.17 (VDD)
- new net: C31.1, D1.4, FB2.1, R32.2
- new net: C9.1, FB2.2, FB203.1
- new net: Q3.1 (B), R2.1, R3.2, U1.18 (DCT2)
- new net: Q3.2 (E), U1.19 (QE), Z1.2 (A)
- new net: C10.2, Q2.1 (B), Q3.3 (C), R6.1
- new net: C4.1, C7.1, R1.1, R10.1
- new net: Q1.2 (E), Q4.3 (C), R10.2, R11.1, R5.1
- new net: R52.2, U2.1 (CS)
- new net: C31.2, R32.1, R33.2
- new net: C10.1, C3.1, D1.1 (+), Q1.3 (C), Q2.2 (E), R6.2
- new net: C32.1, D1.3, FB1.1, R35.2
- new net: R1.2, U1.20 (DCT)
- new net: R34.1, U1.7 (RNG1)
- new net: C32.2, R34.2, R35.1
- new net: R12.1, U2.15 (C1A)
- new net: C1.1, R12.2
- new net: C5.1, U1.6 (VREG)
- new net: C51.1, U2.16 (VA)
- new net: Q1.1 (B), Q2.3 (C), R3.1, R4.2, R5.2, Z1.1 (K)
- new net: C8.1, FB1.2, FB204.1
- new net: R9.1, U1.3 (IB)
- new net: R13.1, U2.14 (C2A)
- new net: C2.1, R13.2
- new net: C6.1, U1.10 (VREG2)
- new net: Q4.2 (E), U1.13 (QE2)
- new net: Q4.1 (B), R4.1, U1.14 (QB)
- new net: Q5.2 (E), U1.15 (DCT3)
- new net: C4.2, U1.2 (RX)
- new net: C1.2, U1.4 (C1B)
- new net: C2.2, U1.5 (C2B)
- new net: R33.1, U1.9 (RNG2)
- new net: R53.2, U2.2 (FSYNC)
- new net: Q5.1 (B), R2.2
- new net: Q5.3 (C), R11.2
Other:
- note added: "No Ground in DAA Area"
- note removed: "DIGITAL SIDE"
- note removed: "ISOLATION BARRIER"
- note removed: "LINE SIDE"
- note removed: "TELEPHONE LINE"
- moved on the sheet: RV1

Commit message: esp e usb
Parts:
- added C52: 0.1uF, symbol Device:C
- added C75: 10uF, symbol Device:C
- added C76: 22uF, symbol Device:C
- added J2: RJ11, symbol Connector:RJ11
- added J4: USB_C_Receptacle_USB2.0_14P, symbol Connector:USB_C_Receptacle_USB2.0_14P
- added L1: 2.2uH, symbol Device:L
- added R54: 47k Ohm, symbol Device:R
- added R55: 10k Ohm, symbol Device:R
- added R71, R72: 5.1k Ohm, symbol Device:R
- added R73, R74: 22 Ohm, symbol Device:R
- added R75: 100k Ohm, symbol Device:R
- added U3: ESP32-C3-WROOM-02U, RF_Module:ESP32-C3-WROOM-02U, symbol RF_Module:ESP32-C3-WROOM-02U
- added U4: TPS62162DSG, Package_SON:Texas_DSG0008A_WSON-8-1EP_2x2mm_P0.5mm_EP0.9x1.6mm_ThermalVias, symbol Regulator_Switching:TPS62162DSG
- renumbered J2 to J1
Connections:
- net GND: now also C50.1, C52.1, C75.2, C76.2, J4.A1 (GND), J4.A12 (GND), J4.B1 (GND), J4.B12 (GND), R71.2, R72.2, U3.19 (GND), U3.9 (GND), U4.1 (PGND), U4.4 (AGND), U4.5 (FB), U4.9 (PAD); no longer C50.2
- net RING: now also J2.2
- net TIP: now also J2.1
- net CS: now reaches R52.2, U2.1 (CS)
- net CS: now also U3.10 (IO10)
- net FSYNC: now reaches R53.2, U2.2 (FSYNC)
- net FSYNC: now also U3.17 (IO1)
- net RESET: now reaches U2.13 (RESET)
- net RESET: now also R54.2, U3.4 (IO5)
- net SCLK: now reaches U2.19 (SCLK)
- net SCLK: now also U3.5 (IO6)
- net SDO: now reaches U2.23 (SDO)
- net SDO: now also U3.16 (IO2)
- net SDI: now reaches U2.24 (SDI)
- net SDI: now also U3.6 (IO7)
- net PCLK: now reaches U2.3 (PCLK)
- net PCLK: now also U3.18 (IO0)
- net DTX: now reaches U2.4 (DTX)
- net DTX: now also U3.15 (IO3)
- net DRX: now reaches U2.5 (DRX)
- net DRX: now also U3.3 (IO4)
- net VDD renamed +3.3V
- net +3.3V: now also C50.2, C76.1, L1.1, R54.1, R55.1, R75.1, U3.1 (3V3), U4.6 (VOS); no longer C50.1
- new net: J4.B7 (D-), R73.1
- new net: R73.2, U3.13 (IO18)
- new net: C75.1, J4.A4 (VBUS), J4.A9 (VBUS), J4.B4 (VBUS), J4.B9 (VBUS), U4.2 (VIN), U4.3 (EN)
- new net: L1.2, U4.7 (SW)
- new net: R75.2, U4.8 (PG)
- new net: J4.A6 (D+), R74.1
- new net: R74.2, U3.14 (IO19)
- new net: J4.A5 (CC1), R71.1
- new net: J4.B5 (CC2), R72.1
- new net: C52.2, R55.2, U3.2 (EN)
Other:
- moved on the sheet: C1, C2, C50, C51, J1, R12, R13, R52, R53, U2

Commit message: terminando schematic
Parts:
- added C_LED: 100nF, symbol Device:C
- added D2: WS2812B-2020, LED_SMD:LED_WS2812B-2020_PLCC4_2.0x2.0mm, symbol LED:WS2812B-2020
- added R_LED: 330 Ohm, symbol Device:R
- added R_bot: 10k Ohm, symbol Device:R
- added SW1: SW_MEC_5E, symbol Switch:SW_MEC_5E
- renumbered C32 to C30, R35 to R30, R34 to R31
Connections:
- net +3.3V: now also R_bot.1
- net GND: now also C_LED.2, D2.2 (VSS), SW1.4 (A)
- net QE: now reaches Q3.2 (E), U1.19 (QE), Z1.2 (A)
- net RNG1: now reaches R31.1, U1.7 (RNG1)
- net at C75.1, J4.A4 (VBUS), J4.A9 (VBUS)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: now also C_LED.1, D2.4 (VDD)
- net QE2: now reaches Q4.2 (E), U1.13 (QE2)
- net QB: now reaches Q4.1 (B), R4.1, U1.14 (QB)
- net DCT3: now reaches Q5.2 (E), U1.15 (DCT3)
- net RNG2: now reaches R33.1, U1.9 (RNG2)
- net at U3.11 (IO20/RXD): now also R_bot.2, SW1.1
- net at U3.12 (IO21/TXD): now also R_LED.1
- new net: D2.3 (DIN), R_LED.2
- no-connect marks 0 -> 1
Other:
- moved on the sheet: C5, C6, R1

Commit message: edit esp
Parts:
- removed U3: ESP32-C3-WROOM-02U, RF_Module:ESP32-C3-WROOM-02U, symbol RF_Module:ESP32-C3-WROOM-02U
- added U5: ESP32-C3-WROOM-02, RF_Module:ESP32-C3-WROOM-02, symbol RF_Module:ESP32-C3-WROOM-02
Connections:
- net +3.3V: now also U5.1 (3V3)
- net CS: now also U5.10 (IO10)
- net DRX: now also U5.3 (IO4)
- net DTX: now also U5.15 (IO3)
- net FSYNC: now also U5.17 (IO1)
- net GND: now also U5.19 (GND), U5.9 (GND)
- net PCLK: now also U5.18 (IO0)
- net RESET: now also U5.4 (IO5)
- net SCLK: now also U5.5 (IO6)
- net SDI: now also U5.6 (IO7)
- net SDO: now also U5.16 (IO2)
- net at R73.2: now also U5.13 (IO18)
- net at R74.2: now also U5.14 (IO19)
- net at C52.2, R55.2: now also U5.2 (EN)
- net at R_bot.2, SW1.1: now also U5.11 (IO20/RXD)
- net at R_LED.1: now also U5.12 (IO21/TXD)
Changed lines of the file:
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@@
 	)
 	(junction
-		(at 123.19 85.09)
-		(diameter 0)
-		(color 0 0 0 0)
-	)
-	(junction
 		(at 69.85 95.25)
 		(diameter 0)
@@
 		(color 0 0 0 0)
 	)
+	(junction
+		(at 123.19 85.09)
+		(diameter 0)
+		(color 0 0 0 0)
+	)
 	(no_connect
 		(at 96.52 149.86)
@@
 	)
 	(symbol
+		(lib_id "RF_Module:ESP32-C3-WROOM-02")
+		(at 107.95 102.87 0)
+		(unit 1)
+		(body_style 1)
+		(exclude_from_sim no)
+		(in_bom yes)
+		(on_board yes)
+		(in_pos_files yes)
+		(dnp no)
+		(fields_autoplaced yes)
+		(property "Reference" "U5"
+			(at 110.0933 77.47 0)
+			(show_name no)
+			(do_not_autoplace no)
+			(effects
+				(font
+					(size 1.27 1.27)
+				)
+				(justify left)
+			)
+		)
+		(property "Value" "ESP32-C3-WROOM-02"
+			(at 110.0933 80.01 0)
+			(show_name no)
+			(do_not_autoplace no)
+			(effects
+				(font
+					(size 1.27 1.27)
+				)
+				(justify left)
+			)
+		)
+		(property "Footprint" "RF_Module:ESP32-C3-WROOM-02"
+			(at 107.95 102.235 0)
+			(hide yes)
+			(show_name no)
+			(do_not_autoplace no)
+			(effects
+				(font
+					(size 1.27 1.27)
+				)
+			)
+		)
+		(property "Datasheet" "https://www.espressif.com/sites/default/files/documentation/esp32-c3-wroom-02_datasheet_en.pdf"
+			(at 107.95 102.235 0)
+			(hide yes)
+			(show_name no)
+			(do_not_autoplace no)
+			(effects
+				(font
+					(size 1.27 1.27)
+				)
+			)
+		)
+		(property "Description" "802.11 b/g/n Wi­Fi and Bluetooth 5 module, ESP32­C3 SoC, RISC­V microprocessor, On-board antenna"
+			(at 107.95 102.235 0)
+			(hide yes)
+			(show_name no)
+			(do_not_autoplace no)
+			(effects
+				(font
+					(size 1.27 1.27)
+				)
+			)
+		)
+		(pin "8"
+		)
+		(pin "3"
+		)
+		(pin "5"
+		)
+		(pin "13"
+		)
+		(pin "11"
+		)
+		(pin "4"
+		)
+		(pin "6"
+		)
+		(pin "9"
+		)
+		(pin "12"
+		)
+		(pin "14"
+		)
+		(pin "2"
+		)
+		(pin "16"
+		)
+		(pin "7"
+		)
+		(pin "1"
+		)
+		(pin "15"
+		)
+		(pin "17"
+		)
+		(pin "18"
+		)
+		(pin "10"
+		)
+		(pin "19"
+		)
+		(instances
+			(project "interhardware"
+				(path "/54dcf537-a517-4a60-ba81-f3f59fcd6b9a"
+					(reference "U5")
+					(unit 1)
+				)
+			)
+		)
+	)
+	(symbol
 		(lib_id "Transistor_BJT:MMBTA42")
 		(at 351.79 85.09 270)
@@
 					(unit 1)
 				)
-			)
-		)
-	)
-	(symbol
-		(lib_id "RF_Module:ESP32-C3-WROOM-02U")
-		(at 107.95 102.87 0)
-		(unit 1)
-		(body_style 1)
-		(exclude_from_sim no)
-		(in_bom yes)
-		(on_board yes)
-		(in_pos_files yes)
-		(dnp no)
-		(property "Reference" "U3"
-			(at 110.0933 77.47 0)
-			(show_name no)
-			(do_not_autoplace no)
-			(effects
-				(font
-					(size 1.27 1.27)
-				)
-				(justify left)
-			)
-		)
-		(property "Value" "ESP32-C3-WROOM-02U"
-			(at 110.0933 80.01 0)
-			(show_name no)
-			(do_not_autoplace no)
-			(effects
-				(font
-					(size 1.27 1.27)
-				)
-				(justify left)
-			)
-		)
-		(property "Footprint" "RF_Module:ESP32-C3-WROOM-02U"
-			(at 107.95 103.505 0)
-			(hide yes)
-			(show_name no)
-			(do_not_autoplace no)
-			(effects
-				(font
-					(size 1.27 1.27)
-				)
-			)
-		)
-		(property "Datasheet" "https://www.espressif.com/sites/default/files/documentation/esp32-c3-wroom-02_datasheet_en.pdf"
-			(at 107.95 103.505 0)
-			(hide yes)
-			(show_name no)
-			(do_not_autoplace no)
-			(effects
-				(font
-					(size 1.27 1.27)
-				)
-			)
-		)
-		(property "Description" "802.11 b/g/n Wi­Fi and Bluetooth 5 module, ESP32­C3 SoC, RISC­V microprocessor, On-board antenna"
-			(at 107.95 103.505 0)
-			(hide yes)
-			(show_name no)
-			(do_not_autoplace no)
-			(effects
-				(font
-					(size 1.27 1.27)
-				)
-			)
-		)
-		(pin "15"
-		)
-		(pin "12"
-		)
-		(pin "6"
-		)
-		(pin "13"
-		)
-		(pin "9"
-		)
-		(pin "14"
-		)
-		(pin "5"
-		)
-		(pin "1"
-		)
-		(pin "2"
-		)
-		(pin "8"
-		)
-		(pin "19"
-		)
-		(pin "10"
-		)
-		(pin "7"
-		)
-		(pin "3"
-		)
-		(pin "4"
-		)
-		(pin "11"
-		)
-		(pin "16"
-		)
-		(pin "18"
-		)
-		(pin "17"
-		)
-		(instances
-			(project "interhardware"
-				(path "/54dcf537-a517-4a60-ba81-f3f59fcd6b9a"
-					(reference "U3")
-					(unit 1)
-				)

Commit message: footprints iniciais
Parts:
- removed SW1: SW_MEC_5E, symbol Switch:SW_MEC_5E
- added SW1: SW_Omron_B3FS, Button_Switch_SMD:SW_SPST_B3U-1000P, symbol Switch:SW_Omron_B3FS
- C50, C51, C52: footprint (none) -> Capacitor_SMD:C_0603_1608Metric
- C_LED: value 100nF -> 0.1uF; footprint (none) -> Capacitor_SMD:C_0603_1608Metric
- J1, J2: footprint (none) -> Connector_RJ:RJ12_Amphenol_54601-x06_Horizontal
- J4: footprint (none) -> Connector_USB:USB_C_Receptacle_GCT_USB4105-xx-A_16P_TopMnt_Horizontal
- R52, R53, R54, R55, R71, R72, R73, R74, R75, R_LED, R_bot: footprint (none) -> Resistor_SMD:R_0603_1608Metric
- U1: footprint (none) -> interbridge_telephony:3019-F-FM-QFN40P300X300X90-21N
- U2: footprint (none) -> interbridge_telephony:3050-E1-FM-QFN50P400X400X80-25N
Connections:
- net GND: now also SW1.2
- net at R_bot.2, U5.11 (IO20/RXD): now also SW1.1
Changed lines of the file:
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@@
 			)
 		)
-		(property "Footprint" ""
+		(property "Footprint" "Resistor_SMD:R_0603_1608Metric"
 			(at 144.018 74.93 90)
 			(hide yes)
@@
 			)
 		)
-		(property "Footprint" ""
+		(property "Footprint" "Resistor_SMD:R_0603_1608Metric"
 			(at 80.01 119.888 90)
 			(hide yes)
@@
 			)
 		)
-		(property "Footprint" ""
+		(property "Footprint" "Capacitor_SMD:C_0603_1608Metric"
 			(at 173.6852 139.7 0)
 			(hide yes)
@@
 			)
 		)
-		(property "Footprint" ""
+		(property "Footprint" "Connector_RJ:RJ12_Amphenol_54601-x06_Horizontal"
 			(at 398.78 186.055 90)
 			(hide yes)
@@
 			)
 		)
-		(property "Footprint" ""
+		(property "Footprint" "Capacitor_SMD:C_0603_1608Metric"
 			(at 166.37 68.2752 0)
 			(hide yes)
@@
 			)
 		)
-		(property "Footprint" ""
+		(property "Footprint" "interbridge_telephony:3019-F-FM-QFN40P300X300X90-21N"
 			(at 238.76 129.54 0)
 			(hide yes)
@@
 			)
 		)
-		(property "Footprint" ""
+		(property "Footprint" "Resistor_SMD:R_0603_1608Metric"
 			(at 80.01 118.872 90)
 			(hide yes)
@@
 			)
 		)
-		(property "Footprint" ""
+		(property "Footprint" "Resistor_SMD:R_0603_1608Metric"
 			(at 54.61 106.172 90)
 			(hide yes)
@@
 			)
 		)
-		(property "Footprint" ""
+		(property "Footprint" "Resistor_SMD:R_0603_1608Metric"
 			(at 188.468 74.93 90)
 			(hide yes)
@@
 			)
 		)
-		(property "Footprint" ""
+		(property "Footprint" "Connector_USB:USB_C_Receptacle_GCT_USB4105-xx-A_16P_TopMnt_Horizontal"
 			(at 29.21 118.11 0)
 			(hide yes)
@@
 			)
 		)
-		(property "Footprint" ""
+		(property "Footprint" "Resistor_SMD:R_0603_1608Metric"
 			(at 54.61 112.268 90)
 			(hide yes)
@@
 			)
 		)
-		(property "Footprint" ""
+		(property "Footprint" "Capacitor_SMD:C_0603_1608Metric"
 			(at 87.63 84.1248 0)
 			(hide yes)
@@
 			)
 		)
-		(property "Footprint" ""
+		(property "Footprint" "Resistor_SMD:R_0603_1608Metric"
 			(at 34.798 57.15 90)
 			(hide yes)
@@
 			)
 		)
-		(property "Footprint" ""
+		(property "Footprint" "Resistor_SMD:R_0603_1608Metric"
 			(at 134.112 67.31 90)
 			(hide yes)
@@
 			)
 		)
-		(property "Footprint" ""
+		(property "Footprint" "Resistor_SMD:R_0603_1608Metric"
 			(at 91.948 64.77 90)
 			(hide yes)
@@
 			)
 		)
-		(property "Footprint" ""
+		(property "Footprint" "Connector_RJ:RJ12_Amphenol_54601-x06_Horizontal"
 			(at 398.78 211.455 90)
 			(hide yes)
@@
 	)
 	(symbol
+		(lib_id "Switch:SW_Omron_B3FS")
+		(at 137.16 116.84 0)
+		(unit 1)
+		(body_style 1)
+		(exclude_from_sim no)
+		(in_bom yes)
+		(on_board yes)
+		(in_pos_files yes)
+		(dnp no)
+		(property "Reference" "SW1"
+			(at 137.16 109.22 0)
+			(show_name no)
+			(do_not_autoplace no)
+			(effects
+				(font
+					(size 1.27 1.27)
+				)
+			)
+		)
+		(property "Value" "SW_Omron_B3FS"
+			(at 134.112 105.664 0)
+			(hide yes)
+			(show_name no)
+			(do_not_autoplace no)
+			(effects
+				(font
+					(size 1.27 1.27)
+				)
+			)
+		)
+		(property "Footprint" "Button_Switch_SMD:SW_SPST_B3U-1000P"
+			(at 137.16 111.76 0)
+			(hide yes)
+			(show_name no)
+			(do_not_autoplace no)
+			(effects
+				(font
+					(size 1.27 1.27)
+				)
+			)
+		)
+		(property "Datasheet" "https://omronfs.omron.com/en_US/ecb/products/pdf/en-b3fs.pdf"
+			(at 137.16 111.76 0)
+			(hide yes)
+			(show_name no)
+			(do_not_autoplace no)
+			(effects
+				(font
+					(size 1.27 1.27)
+				)
+			)
+		)
+		(property "Description" "Omron B3FS 6x6mm single pole normally-open tactile switch"
+			(at 137.16 116.84 0)
+			(hide yes)
+			(show_name no)
+			(do_not_autoplace no)
+			(effects
+				(font
+					(size 1.27 1.27)
+				)
+			)
+		)
+		(pin "2"
+		)
+		(pin "1"
+		)
+		(instances
+			(project "interhardware"
+				(path "/54dcf537-a517-4a60-ba81-f3f59fcd6b9a"
+					(reference "SW1")
+					(unit 1)
+				)
+			)
+		)
+	)
+	(symbol
 		(lib_id "power:+3.3V")
 		(at 62.23 48.26 0)
@@
 			)
 		)
-		(property "Footprint" ""
+		(property "Footprint" "Resistor_SMD:R_0603_1608Metric"
 			(at 124.968 72.39 90)
 			(hide yes)
@@
 			)
 		)
-		(property "Footprint" ""
+		(property "Footprint" "Resistor_SMD:R_0603_1608Metric"
 			(at 121.412 127 90)
 			(hide yes)
@@
 			)
 		)
-		(property "Value" "100nF"
+		(property "Value" "0.1uF"
 			(at 97.7899 158.75 0)
 			(show_name no)
@@
 			)
 		)
-		(property "Footprint" ""
+		(property "Footprint" "Capacitor_SMD:C_0603_1608Metric"
 			(at 100.33 155.9052 0)
 			(hide yes)
@@
 	)
 	(symbol
-		(lib_id "Switch:SW_MEC_5E")
-		(at 137.16 119.38 0)
-		(unit 1)
-		(body_style 1)
-		(exclude_from_sim no)
-		(in_bom yes)
-		(on_board yes)
-		(in_pos_files yes)
-		(dnp no)
-		(fields_autoplaced yes)
-		(property "Reference" "SW1"
-			(at 137.16 109.22 0)
-			(show_name no)
-			(do_not_autoplace no)
-			(effects
-				(font
-					(size 1.27 1.27)
-				)
-			)
-		)
-		(property "Value" "SW_MEC_5E"
-			(at 137.16 111.76 0)
-			(show_name no)
-			(do_not_autoplace no)
-			(effects
-				(font
-					(size 1.27 1.27)
-				)
-			)
-		)
-		(property "Footprint" ""
-			(at 137.16 111.76 0)
-			(hide yes)
-			(show_name no)
-			(do_not_autoplace no)
-			(effects
-				(font
-					(size 1.27 1.27)
-				)
-			)
-		)
-		(property "Datasheet" "https://www.apem.com/medias/download/MEC_switches_serie_MULTIMEC5E.pdf"
-			(at 137.16 111.76 0)
-			(hide yes)
-			(show_name no)
-			(do_not_autoplace no)
-			(effects
-				(font
-					(size 1.27 1.27)
-				)
-			)
-		)
-		(property "Description" "MEC 5E single pole normally-open tactile switch"
-			(at 137.16 119.38 0)
-			(hide yes)
-			(show_name no)
-			(do_not_autoplace no)
-			(effects
-				(font
-					(size 1.27 1.27)
-				)
-			)
-		)
-		(pin "3"
-		)
-		(pin "1"
-		)
-		(pin "2"
-		)
-		(pin "4"
-		)
-		(instances
-			(project "interhardware"
-				(path "/54dcf537-a517-4a60-ba81-f3f59fcd6b9a"
-					(reference "SW1")
-					(unit 1)
-				)
-			)
-		)
-	)
-	(symbol
 		(lib_id "interbridge_telephony:SI3050-E1-FM")
 		(at 165.1 102.87 0)
@@
 			)
 		)
-		(property "Footprint" ""
+		(property "Footprint" "interbridge_telephony:3050-E1-FM-QFN50P400X400X80-25N"
 			(at 165.1 102.87 0)
 			(hide yes)
