File: kicad/interhardware.kicad_sch (KiCad schematic)
At the start: 65 parts, among them J1 RJE0166002, J2 USB_C_Receptacle_USB2.0_16P, Q1 MMBTA42, Q2 MMBTA92, Q3 MMBTA42, Q4 MMBTA06, Q5 MMBTA06, SW1 B3U-1000P, U3 ESP32-C3-WROOM-02, U4 TPS62162DSG

Commit message: finalize MDB6S procurement release artifacts
Parts:
- D1: MPN (none) -> MDB6S; Manufacturer (none) -> onsemi; Package (none) -> TSSOP-4 / MDBxS
Changed lines of the file:
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@@
 			)
 		)
-		(property "Description" "Single-Phase Bridge Rectifier, 420V Vrms, 1A If, TSSOP-4"
+		(property "Description" "1 A, 600 V single-phase bridge rectifier"
 			(at 321.31 186.69 0)
 			(hide yes)
 			(show_name no)
+			(do_not_autoplace no)
+			(effects
+				(font
+					(size 1.27 1.27)
+				)
+			)
+		)
+		(property "Manufacturer" "onsemi"
+			(at 0 0 0)
+			(hide yes)
+			(show_name no)
+			(do_not_autoplace no)
+			(effects
+				(font
+					(size 1.27 1.27)
+				)
+			)
+		)
+		(property "MPN" "MDB6S"
+			(at 0 0 0)
+			(hide yes)
+			(show_name no)
+			(do_not_autoplace no)
+			(effects
+				(font
+					(size 1.27 1.27)
+				)
+			)
+		)
+		(property "Package" "TSSOP-4 / MDBxS"
+			(at 0 0 0)
+			(hide yes)
+			(show_name no)

Commit message: nova forma e usando gpio8
Parts:
- added EN, J3, J4: Conn_01x01, Connector_PinHeader_2.54mm:PinHeader_1x01_P2.54mm_Vertical, symbol Connector_Generic:Conn_01x01
- added R56, R57: 10k Ohm, Resistor_SMD:R_0603_1608Metric, symbol Device:R
Connections:
- net +3.3V: now also R56.1, R57.1; no longer R54.1
- net GND: now also R54.2, J4.1 (Pin_1)
- net RESET: now also R54.1; no longer R54.2
- net SDO: now also R56.2
- net RGDT: now reaches U2.6 (RGDT)
- net RGDT: now also U3.7 (IO8)
- net EN: now reaches C52.2, R55.2, U3.2 (EN)
- net EN: now also EN.1 (Pin_1)
- net BOOT: now reaches U3.8 (IO9)
- net BOOT: now also J3.1 (Pin_1), R57.2
- no-connect marks 19 -> 16
Other:
- moved on the sheet: R54, R55, SW1

Commit message: maisum pad
Parts:
- added AOUT1: Conn_01x01, Connector_PinHeader_2.54mm:PinHeader_1x01_P2.54mm_Vertical, symbol Connector_Generic:Conn_01x01
- renumbered J3 to BOOT1, EN to EN1, J4 to GND1
Connections:
- net at U2.7 (AOUT/INT): now also AOUT1.1 (Pin_1)
- no-connect marks 16 -> 15
Changed lines of the file:
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@@
 	)
 	(no_connect
-		(at 153.67 111.76)
-	)
-	(no_connect
 		(at 96.52 149.86)
 	)
@@
 	(wire
 		(pts
+			(xy 148.59 124.46) (xy 148.59 111.76)
+		)
+		(stroke
+			(width 0)
+			(type default)
+		)
+	)
+	(wire
+		(pts
 			(xy 172.72 132.08) (xy 172.72 129.54)
 		)
@@
 	(wire
 		(pts
+			(xy 148.59 111.76) (xy 153.67 111.76)
+		)
+		(stroke
+			(width 0)
+			(type default)
+		)
+	)
+	(wire
+		(pts
 			(xy 328.93 186.69) (xy 328.93 158.75)
 		)
@@
 		(dnp no)
 		(fields_autoplaced yes)
-		(property "Reference" "J4"
+		(property "Reference" "GND1"
 			(at 152.4 134.6199 0)
 			(show_name no)
@@
 			(project "interhardware"
 				(path "/54dcf537-a517-4a60-ba81-f3f59fcd6b9a"
-					(reference "J4")
+					(reference "GND1")
 					(unit 1)
 				)
@@
 	)
 	(symbol
+		(lib_id "Connector_Generic:Conn_01x01")
+		(at 148.59 129.54 270)
+		(unit 1)
+		(body_style 1)
+		(exclude_from_sim no)
+		(in_bom yes)
+		(on_board yes)
+		(in_pos_files yes)
+		(dnp no)
+		(fields_autoplaced yes)
+		(property "Reference" "AOUT1"
+			(at 151.13 128.2699 90)
+			(show_name no)
+			(do_not_autoplace no)
+			(effects
+				(font
+					(size 1.27 1.27)
+				)
+				(justify left)
+			)
+		)
+		(property "Value" "Conn_01x01"
+			(at 151.13 130.8099 90)
+			(show_name no)
+			(do_not_autoplace no)
+			(effects
+				(font
+					(size 1.27 1.27)
+				)
+				(justify left)
+			)
+		)
+		(property "Footprint" "Connector_PinHeader_2.54mm:PinHeader_1x01_P2.54mm_Vertical"
+			(at 148.59 129.54 0)
+			(hide yes)
+			(show_name no)
+			(do_not_autoplace no)
+			(effects
+				(font
+					(size 1.27 1.27)
+				)
+			)
+		)
+		(property "Datasheet" ""
+			(at 148.59 129.54 0)
+			(hide yes)
+			(show_name no)
+			(do_not_autoplace no)
+			(effects
+				(font
+					(size 1.27 1.27)
+				)
+			)
+		)
+		(property "Description" "Generic connector, single row, 01x01, script generated (kicad-library-utils/schlib/autogen/connector/)"
+			(at 148.59 129.54 0)
+			(hide yes)
+			(show_name no)
+			(do_not_autoplace no)
+			(effects
+				(font
+					(size 1.27 1.27)
+				)
+			)
+		)
+		(pin "1"
+		)
+		(instances
+			(project "interhardware"
+				(path "/54dcf537-a517-4a60-ba81-f3f59fcd6b9a"
+					(reference "AOUT1")
+					(unit 1)
+				)
+			)
+		)
+	)
+	(symbol
 		(lib_id "Transistor_BJT:MMBTA06")
 		(at 302.26 109.22 0)
@@
 		(dnp no)
 		(fields_autoplaced yes)
-		(property "Reference" "J3"
+		(property "Reference" "BOOT1"
 			(at 123.19 46.9899 0)
 			(show_name no)
@@
 			(project "interhardware"
 				(path "/54dcf537-a517-4a60-ba81-f3f59fcd6b9a"
-					(reference "J3")
+					(reference "BOOT1")
 					(unit 1)
 				)
@@
 		(dnp no)
 		(fields_autoplaced yes)
-		(property "Reference" "EN"
+		(property "Reference" "EN1"
 			(at 95.25 46.9899 0)
 			(show_name no)
@@
 			(project "interhardware"
 				(path "/54dcf537-a517-4a60-ba81-f3f59fcd6b9a"
-					(reference "EN")
+					(reference "EN1")
 					(unit 1)
 				)

Commit message: ajuste chek-up
Parts:
- added R58: 4.7k Ohm, Resistor_SMD:R_0603_1608Metric, symbol Device:R
- R54: value 47k Ohm -> 10k Ohm
Connections:
- net +3.3V: now also R58.1
- net RGDT: now also R58.2
Other:
- moved on the sheet: BOOT1, R57
Changed lines of the file:
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@@
 	)
 	(junction
+		(at 87.63 35.56)
+		(diameter 0)
+		(color 0 0 0 0)
+	)
+	(junction
 		(at 74.93 35.56)
 		(diameter 0)
@@
 	)
 	(junction
-		(at 87.63 35.56)
-		(diameter 0)
-		(color 0 0 0 0)
-	)
-	(junction
-		(at 115.57 48.26)
+		(at 110.49 48.26)
 		(diameter 0)
 		(color 0 0 0 0)
@@
 	)
 	(junction
+		(at 110.49 35.56)
+		(diameter 0)
+		(color 0 0 0 0)
+	)
+	(junction
 		(at 25.4 140.97)
 		(diameter 0)
@@
 	(wire
 		(pts
+			(xy 110.49 35.56) (xy 132.08 35.56)
+		)
+		(stroke
+			(width 0)
+			(type default)
+		)
+	)
+	(wire
+		(pts
 			(xy 33.02 35.56) (xy 58.42 35.56)
 		)
@@
 	(wire
 		(pts
-			(xy 87.63 35.56) (xy 115.57 35.56)
+			(xy 87.63 35.56) (xy 110.49 35.56)
 		)
 		(stroke
@@
 	(wire
 		(pts
+			(xy 132.08 44.45) (xy 132.08 48.26)
+		)
+		(stroke
+			(width 0)
+			(type default)
+		)
+	)
+	(wire
+		(pts
 			(xy 337.82 153.67) (xy 349.25 153.67)
 		)
@@
 	(wire
 		(pts
+			(xy 132.08 36.83) (xy 132.08 35.56)
+		)
+		(stroke
+			(width 0)
+			(type default)
+		)
+	)
+	(wire
+		(pts
 			(xy 45.72 87.63) (xy 48.26 87.63)
 		)
@@
 	(wire
 		(pts
-			(xy 115.57 36.83) (xy 115.57 35.56)
+			(xy 110.49 36.83) (xy 110.49 35.56)
 		)
 		(stroke
@@
 	(wire
 		(pts
-			(xy 115.57 48.26) (xy 115.57 52.07)
+			(xy 110.49 48.26) (xy 110.49 52.07)
 		)
 		(stroke
@@
 	(wire
 		(pts
-			(xy 115.57 44.45) (xy 115.57 48.26)
+			(xy 110.49 44.45) (xy 110.49 48.26)
 		)
 		(stroke
@@
 		)
 	)
+	(label "RGDT"
+		(at 132.08 48.26 0)
+		(effects
+			(font
+				(size 1.27 1.27)
+			)
+			(justify left bottom)
+		)
+	)
 	(label "DCT3"
 		(at 304.8 135.89 0)
@@
 	)
 	(label "BOOT"
-		(at 115.57 52.07 0)
+		(at 110.49 52.07 0)
 		(effects
 			(font
@@
 	(symbol
 		(lib_id "Device:R")
-		(at 115.57 40.64 0)
+		(at 110.49 40.64 0)
 		(unit 1)
 		(body_style 1)
@@
 		(dnp no)
 		(property "Reference" "R57"
-			(at 113.03 39.3699 0)
+			(at 107.95 39.3699 0)
 			(show_name no)
 			(do_not_autoplace no)
@@
 		)
 		(property "Value" "10k Ohm"
-			(at 113.03 41.9099 0)
+			(at 107.95 41.9099 0)
 			(show_name no)
 			(do_not_autoplace no)
@@
 		)
 		(property "Footprint" "Resistor_SMD:R_0603_1608Metric"
-			(at 113.792 40.64 90)
+			(at 108.712 40.64 90)
 			(hide yes)
 			(show_name no)
@@
 		)
 		(property "Datasheet" ""
-			(at 115.57 40.64 0)
+			(at 110.49 40.64 0)
 			(hide yes)
 			(show_name yes)
@@
 		)
 		(property "Description" "Resistor"
-			(at 115.57 40.64 0)
+			(at 110.49 40.64 0)
 			(hide yes)
 			(show_name no)
@@
 		)
 		(property "Manufacturer" "GENERIC"
-			(at 205.74 -24.13 0)
+			(at 200.66 -24.13 0)
 			(hide yes)
 			(show_name no)
@@
 		)
 		(property "MPN" "GENERIC"
-			(at 205.74 -24.13 0)
+			(at 200.66 -24.13 0)
 			(hide yes)
 			(show_name no)
@@
 		)
 		(property "Package" "0603_1608Metric"
-			(at 205.74 -24.13 0)
+			(at 200.66 -24.13 0)
 			(hide yes)
 			(show_name no)
@@
 	(symbol
 		(lib_id "Connector_Generic:Conn_01x01")
-		(at 120.65 48.26 0)
+		(at 115.57 48.26 0)
 		(unit 1)
 		(body_style 1)
@@
 		(fields_autoplaced yes)
 		(property "Reference" "BOOT1"
-			(at 123.19 46.9899 0)
+			(at 118.11 46.9899 0)
 			(show_name no)
 			(do_not_autoplace no)
@@
 		)
 		(property "Value" "Conn_01x01"
-			(at 123.19 49.5299 0)
+			(at 118.11 49.5299 0)
 			(show_name no)
 			(do_not_autoplace no)
@@
 		)
 		(property "Footprint" "Connector_PinHeader_2.54mm:PinHeader_1x01_P2.54mm_Vertical"
-			(at 120.65 48.26 0)
+			(at 115.57 48.26 0)
 			(hide yes)
 			(show_name no)
@@
 		)
 		(property "Datasheet" ""
-			(at 120.65 48.26 0)
+			(at 115.57 48.26 0)
 			(hide yes)
 			(show_name no)
@@
 		)
 		(property "Description" "Generic connector, single row, 01x01, script generated (kicad-library-utils/schlib/autogen/connector/)"
-			(at 120.65 48.26 0)
+			(at 115.57 48.26 0)
 			(hide yes)
 			(show_name no)
@@
 			)
 		)
-		(property "Value" "47k Ohm"
+		(property "Value" "10k Ohm"
 			(at 142.24 109.2199 0)
 			(show_name no)
@@
 					(unit 1)
 				)
+			)
+		)
+	)
+	(symbol
+		(lib_id "Device:R")
+		(at 132.08 40.64 0)
+		(unit 1)
+		(body_style 1)
+		(exclude_from_sim no)
+		(in_bom yes)
+		(on_board yes)
+		(in_pos_files yes)
+		(dnp no)
+		(property "Reference" "R58"
+			(at 129.54 39.3699 0)
+			(show_name no)
+			(do_not_autoplace no)
+			(effects
+				(font
+					(size 1.27 1.27)
+				)
+				(justify right)
+			)
+		)
+		(property "Value" "4.7k Ohm"
+			(at 129.54 41.9099 0)
+			(show_name no)
+			(do_not_autoplace no)
+			(effects
+				(font
+					(size 1.27 1.27)
+				)
+				(justify right)
+			)
+		)
+		(property "Footprint" "Resistor_SMD:R_0603_1608Metric"
+			(at 130.302 40.64 90)
+			(hide yes)
+			(show_name no)
+			(do_not_autoplace no)
+			(effects
+				(font
+					(size 1.27 1.27)
+				)
+			)
+		)
+		(property "Datasheet" ""
+			(at 132.08 40.64 0)
+			(hide yes)
+			(show_name yes)
+			(do_not_autoplace no)
+			(effects
+				(font
+					(size 1.27 1.27)
+				)
+			)
+		)
+		(property "Description" "Resistor"
+			(at 132.08 40.64 0)
+			(hide yes)
+			(show_name no)
+			(do_not_autoplace no)
+			(effects
+				(font
+					(size 1.27 1.27)
+				)
+			)
+		)
+		(property "Manufacturer" "GENERIC"
+			(at 222.25 -24.13 0)
+			(hide yes)
+			(show_name no)
+			(do_not_autoplace no)
+			(effects
+				(font
+					(size 1.27 1.27)
+				)
+			)
+		)
+		(property "MPN" "GENERIC"
+			(at 222.25 -24.13 0)
+			(hide yes)
+			(show_name no)
+			(do_not_autoplace no)
+			(effects
+				(font
+					(size 1.27 1.27)
+				)
+			)
+		)
+		(property "Package" "0603_1608Metric"
+			(at 222.25 -24.13 0)
+			(hide yes)
+			(show_name no)
+			(do_not_autoplace no)
+			(effects
+				(font
+					(size 1.27 1.27)
+				)
+			)
+		)
+		(pin "1"
+		)
+		(pin "2"
+		)
+		(instances
+			(project "interhardware"
+				(path "/54dcf537-a517-4a60-ba81-f3f59fcd6b9a"
+					(reference "R58")
+					(unit 1)
+				)
