File: kicad/interhardware.kicad_pcb (KiCad board)
At the start: 2 copper layers, 72.2 x 56.2 mm, 65 parts, among them J1 RJE0166002, J2 USB_C_Receptacle_USB2.0_16P, Q1 MMBTA42, Q2 MMBTA92, Q3 MMBTA42, Q4 MMBTA06, Q5 MMBTA06, SW1 B3U-1000P, U3 ESP32-C3-WROOM-02, U4 TPS62162DSG

Commit message: edit pra deixar 100%
Parts:
- moved C75 11.1 mm to (245.7, 92.4), turned to 180 degrees
- moved C76 0.80 mm to (243.6, 89.7)
- moved R74 0.80 mm to (244.8, 94.2)
- moved R_BO1 0.80 mm to (228.2, 94.8)
- moved U4 0.80 mm to (249.0, 90.4)
- moved C52 0.80 mm to (191.0, 93.6)
- moved C_LED1 0.80 mm to (235.2, 99.2)
- moved D2 0.80 mm to (232.1, 99.8)
- moved J2 0.80 mm to (255.9, 95.2)
- moved L1 0.80 mm to (247.4, 86.0)
- moved R52 0.80 mm to (214.5, 102.6)
- moved R53 0.80 mm to (214.8, 92.1)
- moved R55 0.80 mm to (191.0, 92.1)
- moved R71 0.80 mm to (248.8, 96.5)
- moved R72 0.80 mm to (249.0, 93.5)
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Routing:
- net Net-(U3-IO19): track 40.9 -> 33.0 mm, vias 0 -> 2
- net Net-(U3-IO18): track 39.7 -> 33.4 mm, vias 0 -> 2
- net Net-(U3-IO20/RXD): track 23.2 -> 21.6 mm
- net GND: track 186.8 -> 188.2 mm
- net +3.3V: track 134.5 -> 133.1 mm
- net /DRX: track 33.9 -> 33.0 mm
- net /SCLK: track 25.8 -> 25.0 mm
- net /PCLK: track 45.4 -> 44.6 mm
- net /SDI: track 24.8 -> 24.0 mm
- net /RESET: track 39.2 -> 38.4 mm
- net /FSYNC: track 45.1 -> 44.3 mm
- net Net-(U3-IO21/TXD): vias 2 -> 0
Other:
- board size 72.2 x 56.2 mm -> 72 x 55.4 mm

Commit message: ajuste do D1
Parts:
- D1: value MB6S -> MDB6S; footprint Package_TO_SOT_SMD:TO-269AA -> Package_SO:TSSOP-4_4.4x5mm_P4mm
- moved RV1 0.30 mm to (239.8, 119.8)
- moved D1 0.22 mm to (233.3, 119.4)
- moved R13 0.15 mm to (197.6, 123.0)
Connections:
- D1 pad 1: /IGND -> Net-(D1-+)
- D1 pad 2: Net-(Q1-C) -> Net-(D1--)
- D1 pad 3: Net-(D1-+) -> /IGND
- D1 pad 4: Net-(D1--) -> Net-(Q1-C)
Routing:
- net Net-(D1-+): track 31.8 -> 37.8 mm, vias 0 -> 2
- net Net-(Q1-C): track 21.9 -> 27.5 mm
- net /IGND: track 21.1 -> 24.3 mm
- net Net-(D1--): track 32.8 -> 30.6 mm, vias 0 -> 2
- net Net-(RV1-K): track 20.4 -> 21.4 mm

Commit message: manufacturing
Routing:
- net GND: track 188.2 -> 200.1 mm, vias 9 -> 10
- net Net-(D2-VDD): track 33.6 -> 33.5 mm, vias 4 -> 2
- net Net-(U3-IO19): vias 2 -> 0
- net Net-(U3-IO18): vias 2 -> 0

Commit message: caminho relativo
Routing:
- net Net-(C9-Pad1): vias 2 -> 3
Changed lines of the file:
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@@
 		(filling no)
 		(pcbplotparams
-			(layerselection 0x00000000_00000000_55555555_5755f5ff)
+			(layerselection 0x00000000_00000000_55555555_5755757f)
 			(plot_on_all_layers_selection 0x00000000_00000000_00000000_00000000)
 			(disableapertmacros no)
@@
 			(drillshape 0)
 			(scaleselection 1)
-			(outputdirectory "C:/Users/hjca1/KiCad/interhardware/manufacturing/gerbers/")
+			(outputdirectory "../manufacturing/gerbers/")
 		)
 	)
@@
 		(net "Net-(C9-Pad1)")
 	)
+	(via
+		(at 238 115.8)
+		(size 0.6)
+		(drill 0.3)
+		(layers "F.Cu" "B.Cu")
+		(net "Net-(C9-Pad1)")
+	)
 	(segment
-		(start 237.2 131)
-		(end 237.2 129.8)
-		(width 0.381)
+		(start 238 129)
+		(end 238 115.8)
+		(width 0.508)
 		(layer "B.Cu")
 		(net "Net-(C9-Pad1)")
 	)
 	(segment
-		(start 238 115.8)
+		(start 237.2 129.8)
 		(end 238 129)
 		(width 0.508)
@@
 	)
 	(segment
-		(start 237.2 129.8)
-		(end 238 129)
-		(width 0.381)
+		(start 237.2 131)
+		(end 237.2 129.8)
+		(width 0.508)
 		(layer "B.Cu")
 		(net "Net-(C9-Pad1)")

Commit message: nova forma e usando gpio8
Parts:
- added BOOT: Conn_01x01, Connector_PinHeader_2.54mm:PinHeader_1x01_P2.54mm_Vertical, F.Cu at (191.2, 106.2)
- added EN: Conn_01x01, Connector_PinHeader_2.54mm:PinHeader_1x01_P2.54mm_Vertical, F.Cu at (223.0, 88.0)
- added GND: Conn_01x01, Connector_PinHeader_2.54mm:PinHeader_1x01_P2.54mm_Vertical, F.Cu at (226.6, 88.0)
- added R56: 10k Ohm, Resistor_SMD:R_0603_1608Metric, F.Cu at (214.8, 93.6)
- added R57: 10k Ohm, Resistor_SMD:R_0603_1608Metric, F.Cu at (190.4, 101.2)
- moved R55 1.62 mm to (192.6, 92.4), turned to -90 degrees
- moved C52 1.26 mm to (191.1, 92.3), turned to -90 degrees
- moved R54 1.07 mm to (195.8, 125.6), turned to -90 degrees
Connections:
- net Net-(U3-EN) renamed /EN
- R54 pad 1: +3.3V -> /RESET
- R54 pad 2: /RESET -> GND
- U2 pad 6: unconnected-(U2-RGDT-Pad6) -> /RGDT
- U3 pad 7: unconnected-(U3-IO8-Pad7) -> /RGDT
- U3 pad 8: unconnected-(U3-IO9-Pad8) -> /BOOT
Routing:
- net /EN: track 4.30 -> 34.6 mm, vias 0 -> 1
- net /RGDT: track 0.00 -> 30.1 mm, vias 0 -> 2
- net GND: track 200.1 -> 210.5 mm
- net /BOOT: track 0.00 -> 8.32 mm
- net /RESET: track 38.4 -> 35.4 mm
- net /DRX: track 33.0 -> 35.1 mm
- net /SDO: track 34.5 -> 36.1 mm
- net Net-(C9-Pad1): vias 3 -> 2

Commit message: maisum pad
Parts:
- added AOUT: Conn_01x01, Connector_PinHeader_2.54mm:PinHeader_1x01_P2.54mm_Vertical, F.Cu at (190.4, 128.2)
Connections:
- U2 pad 7: unconnected-(U2-AOUT/INT-Pad7) -> Net-(AOUT1-Pin_1)
Routing:
- net Net-(AOUT1-Pin_1): track 0.00 -> 5.90 mm

Commit message: ajuste chek-up
Parts:
- added R58: 4.7k Ohm, Resistor_SMD:R_0603_1608Metric, F.Cu at (191.9, 98.4)
- R54: value 47k Ohm -> 10k Ohm
- renumbered AOUT to AOUT1, BOOT to BOOT1, EN to EN1, GND to GND1
Routing:
- net +3.3V: track 132.7 -> 134.9 mm
- net /RGDT: track 30.1 -> 31.4 mm
Changed lines of the file:
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@@
 		)
 	)
+	(footprint "Resistor_SMD:R_0603_1608Metric"
+		(layer "F.Cu")
+		(at 191.905 98.355)
+		(descr "Resistor SMD 0603 (1608 Metric), square (rectangular) end terminal, IPC-7351 nominal, (Body size source: IPC-SM-782 page 72, https://www.pcb-3d.com/wordpress/wp-content/uploads/ipc-sm-782a_amendment_1_and_2.pdf)")
+		(tags "resistor")
+		(property "Reference" "R58"
+			(at 0 -1.43 0)
+			(layer "F.SilkS")
+			(effects
+				(font
+					(size 1 1)
+					(thickness 0.15)
+				)
+			)
+		)
+		(property "Value" "4.7k Ohm"
+			(at 0 1.43 0)
+			(layer "F.Fab")
+			(hide yes)
+			(effects
+				(font
+					(size 1 1)
+					(thickness 0.15)
+				)
+			)
+		)
+		(property "Datasheet" ""
+			(at 0 0 0)
+			(layer "F.Fab")
+			(hide yes)
+			(effects
+				(font
+					(size 1.27 1.27)
+				)
+			)
+		)
+		(property "Description" "Resistor"
+			(at 0 0 0)
+			(layer "F.Fab")
+			(hide yes)
+			(effects
+				(font
+					(size 1.27 1.27)
+				)
+			)
+		)
+		(property "KiLib_Generator" "SMD_2terminal_chip_molded"
+			(at 0 0 0)
+			(layer "F.SilkS")
+			(hide yes)
+			(effects
+				(font
+					(size 1 1)
+					(thickness 0.15)
+				)
+			)
+		)
+		(property "Manufacturer" "GENERIC"
+			(at 0 0 0)
+			(unlocked yes)
+			(layer "F.Fab")
+			(hide yes)
+			(effects
+				(font
+					(size 1 1)
+					(thickness 0.15)
+				)
+			)
+		)
+		(property "MPN" "GENERIC"
+			(at 0 0 0)
+			(unlocked yes)
+			(layer "F.Fab")
+			(hide yes)
+			(effects
+				(font
+					(size 1 1)
+					(thickness 0.15)
+				)
+			)
+		)
+		(property "Package" "0603_1608Metric"
+			(at 0 0 0)
+			(unlocked yes)
+			(layer "F.Fab")
+			(hide yes)
+			(effects
+				(font
+					(size 1 1)
+					(thickness 0.15)
+				)
+			)
+		)
+		(property ki_fp_filters "R_*")
+		(sheetname "/")
+		(sheetfile "interhardware.kicad_sch")
+		(units
+			(unit
+				(name "A")
+				(pins "1" "2")
+			)
+		)
+		(attr smd)
+		(duplicate_pad_numbers_are_jumpers no)
+		(fp_line
+			(start -0.237258 -0.5225)
+			(end 0.237258 -0.5225)
+			(stroke
+				(width 0.12)
+				(type solid)
+			)
+			(layer "F.SilkS")
+		)
+		(fp_line
+			(start -0.237258 0.5225)
+			(end 0.237258 0.5225)
+			(stroke
+				(width 0.12)
+				(type solid)
+			)
+			(layer "F.SilkS")
+		)
+		(fp_rect
+			(start -1.48 -0.73)
+			(end 1.48 0.73)
+			(stroke
+				(width 0.05)
+				(type solid)
+			)
+			(fill no)
+			(layer "F.CrtYd")
+		)
+		(fp_rect
+			(start -0.8 -0.4125)
+			(end 0.8 0.4125)
+			(stroke
+				(width 0.1)
+				(type solid)
+			)
+			(fill no)
+			(layer "F.Fab")
+		)
+		(fp_text user "${REFERENCE}"
+			(at 0 0 0)
+			(layer "F.Fab")
+			(effects
+				(font
+					(size 0.4 0.4)
+					(thickness 0.06)
+				)
+			)
+		)
+		(pad "1" smd roundrect
+			(at -0.825 0)
+			(size 0.8 0.95)
+			(layers "F.Cu" "F.Mask" "F.Paste")
+			(roundrect_rratio 0.25)
+			(net "+3.3V")
+			(pintype "passive")
+		)
+		(pad "2" smd roundrect
+			(at 0.825 0)
+			(size 0.8 0.95)
+			(layers "F.Cu" "F.Mask" "F.Paste")
+			(roundrect_rratio 0.25)
+			(net "/RGDT")
+			(pintype "passive")
+		)
+		(embedded_fonts no)
+		(model "${KICAD10_3DMODEL_DIR}/Resistor_SMD.3dshapes/R_0603_1608Metric.step"
+			(offset
+				(xyz 0 0 0)
+			)
+			(scale
+				(xyz 1 1 1)
+			)
+			(rotate
+				(xyz 0 0 0)
+			)
+		)
+	)
 	(footprint "Capacitor_SMD:C_0603_1608Metric"
 		(layer "F.Cu")
@@
 		(descr "Through hole straight pin header, 1x01, 2.54mm pitch, single row")
 		(tags "Through hole pin header THT 1x01 2.54mm single row")
-		(property "Reference" "AOUT"
+		(property "Reference" "AOUT1"
 			(at 0 2.6 0)
 			(layer "F.SilkS")
@@
 		(descr "Through hole straight pin header, 1x01, 2.54mm pitch, single row")
 		(tags "Through hole pin header THT 1x01 2.54mm single row")
-		(property "Reference" "BOOT"
+		(property "Reference" "BOOT1"
 			(at 0 -2.38 0)
 			(layer "F.SilkS")
@@
 		(descr "Through hole straight pin header, 1x01, 2.54mm pitch, single row")
 		(tags "Through hole pin header THT 1x01 2.54mm single row")
-		(property "Reference" "GND"
+		(property "Reference" "GND1"
 			(at 0 -2.38 0)
 			(layer "F.SilkS")
@@
 		(descr "Through hole straight pin header, 1x01, 2.54mm pitch, single row")
 		(tags "Through hole pin header THT 1x01 2.54mm single row")
-		(property "Reference" "EN"
+		(property "Reference" "EN1"
 			(at 0 -2.38 0)
 			(layer "F.SilkS")
@@
 			)
 		)
-		(property "Value" "47k Ohm"
+		(property "Value" "10k Ohm"
 			(at 0 1.43 90)
 			(layer "F.Fab")
@@
 	)
 	(segment
+		(start 191.08 98.355)
+		(end 191.08 98.28)
+		(width 0.508)
+		(layer "F.Cu")
+		(net "+3.3V")
+	)
+	(segment
 		(start 243.7 88.6)
 		(end 243.6 88.7)
@@
 	)
 	(segment
+		(start 191.08 98.28)
+		(end 189.6 96.8)
+		(width 0.508)
+		(layer "F.Cu")
+		(net "+3.3V")
+	)
+	(segment
 		(start 231.575 88.7)
 		(end 227.275 93)
@@
 	)
 	(segment
+		(start 192.8 98.425)
+		(end 192.73 98.355)
+		(width 0.381)
+		(layer "F.Cu")
+		(net "/RGDT")
+	)
+	(segment
 		(start 192.8 99.6)
 		(end 192.9 99.5)
 		(width 0.381)
 		(layer "F.Cu")
+		(net "/RGDT")
+	)
+	(segment
+		(start 192.8 99.6)
+		(end 192.8 98.425)
+		(width 0.381)
+		(layer "F.Cu")
